File: keyboard2.sch (KiCad schematic (older format))
At the start: 138 parts, among them J1 Conn_01x16_Female, J2 Conn_01x12_Female, K00 KEYSW, K01 KEYSW, K010 KEYSW, K011 KEYSW, K012 KEYSW, K013 KEYSW, K014 KEYSW, K02 KEYSW, K03 KEYSW, K04 KEYSW, K05 KEYSW, K06 KEYSW, K07 KEYSW, K08 KEYSW, K09 KEYSW, K10 KEYSW, K11 KEYSW, K110 KEYSW, K111 KEYSW, K112 KEYSW, K113 KEYSW, K114 KEYSW, K12 KEYSW, K13 KEYSW, K14 KEYSW, K15 KEYSW, K16 KEYSW, K17 KEYSW, K18 KEYSW, K19 KEYSW, K20 KEYSW, K21 KEYSW, K210 KEYSW, K211 KEYSW, K212 KEYSW, K214 KEYSW, K22 KEYSW, K23 KEYSW, K24 KEYSW, K25 KEYSW, K26 KEYSW, K27 KEYSW, K28 KEYSW, K29 KEYSW, K30 KEYSW, K31 KEYSW, K310 KEYSW, K311 KEYSW, K313 KEYSW, K314 KEYSW, K32 KEYSW, K33 KEYSW, K34 KEYSW, K35 KEYSW, K36 KEYSW, K37 KEYSW, K38 KEYSW, K39 KEYSW, K40 KEYSW, K41 KEYSW, K410 KEYSW, K411 KEYSW, K412 KEYSW, K413 KEYSW, K414 KEYSW, K42 KEYSW, K45 KEYSW, K49 KEYSW

Commit message: start work on traces
Parts:
- J1: footprint Connector_PinHeader_1.00mm:PinHeader_1x16_P1.00mm_Vertical -> Connector_PinSocket_1.00mm:PinSocket_1x16_P1.00mm_Vertical
- J2: footprint Connector_PinHeader_1.00mm:PinHeader_1x12_P1.00mm_Vertical -> Connector_PinSocket_1.00mm:PinSocket_1x12_P1.00mm_Vertical
Changed lines of the file:
@@
 F 0 "J2" H 10292 5575 50  0000 C CNN
 F 1 "Conn_01x12_Female" H 10292 5666 50  0000 C CNN
-F 2 "Connector_PinHeader_1.00mm:PinHeader_1x12_P1.00mm_Vertical" H 10400 6400 50  0001 C CNN
+F 2 "Connector_PinSocket_1.00mm:PinSocket_1x12_P1.00mm_Vertical" H 10400 6400 50  0001 C CNN
 F 3 "~" H 10400 6400 50  0001 C CNN
 	1    10400 6400
@@
 F 0 "J1" H 9750 6450 50  0000 L CNN
 F 1 "Conn_01x16_Female" V 9750 5600 50  0000 L CNN
-F 2 "Connector_PinHeader_1.00mm:PinHeader_1x16_P1.00mm_Vertical" H 9700 6300 50  0001 C CNN
+F 2 "Connector_PinSocket_1.00mm:PinSocket_1x16_P1.00mm_Vertical" H 9700 6300 50  0001 C CNN
 F 3 "~" H 9700 6300 50  0001 C CNN
 	1    9700 6300
