File: keyboard2.sch (KiCad schematic (older format))
At the start: 138 parts, among them J1 Conn_01x16_Female, J2 Conn_01x12_Female, K00 KEYSW, K01 KEYSW, K010 KEYSW, K011 KEYSW, K012 KEYSW, K013 KEYSW, K014 KEYSW, K02 KEYSW, K03 KEYSW, K04 KEYSW, K05 KEYSW, K06 KEYSW, K07 KEYSW, K08 KEYSW, K09 KEYSW, K10 KEYSW, K11 KEYSW, K110 KEYSW, K111 KEYSW, K112 KEYSW, K113 KEYSW, K114 KEYSW, K12 KEYSW, K13 KEYSW, K14 KEYSW, K15 KEYSW, K16 KEYSW, K17 KEYSW, K18 KEYSW, K19 KEYSW, K20 KEYSW, K21 KEYSW, K210 KEYSW, K211 KEYSW, K212 KEYSW, K214 KEYSW, K22 KEYSW, K23 KEYSW, K24 KEYSW, K25 KEYSW, K26 KEYSW, K27 KEYSW, K28 KEYSW, K29 KEYSW, K30 KEYSW, K31 KEYSW, K310 KEYSW, K311 KEYSW, K313 KEYSW, K314 KEYSW, K32 KEYSW, K33 KEYSW, K34 KEYSW, K35 KEYSW, K36 KEYSW, K37 KEYSW, K38 KEYSW, K39 KEYSW, K40 KEYSW, K41 KEYSW, K410 KEYSW, K411 KEYSW, K412 KEYSW, K413 KEYSW, K414 KEYSW, K42 KEYSW, K45 KEYSW, K49 KEYSW

Commit message: finished alphanumeric placement on pcb
Parts:
- added D48: D, Diode_SMD:D_SOD-123, symbol Device:D
- added K48: KEYSW, Button_Switch_Keyboard:SW_Cherry_MX_1.25u_PCB, symbol keyboard2-rescue:KEYSW-keyboard_parts
- D01, D010, D011, D012, D013, D014, D02, D03, D04, D05, D06, D07, D08, D09, D10, D11, D110, D111, D112, D113, D114, D12, D13, D14, D15, D16, D17, D18, D19, D20, D21, D210, D211, D212, D214, D22, D23, D24, D25, D26, D27, D28, D29, D30, D31, D310, D311, D313, D314, D32, D33, D34, D35, D36, D37, D38, D39, D40, D41, D410, D411, D412, D413, D414, D42, D45, D49: footprint keyboard_parts:D_SOD123_axial -> Diode_SMD:D_SOD-123
- K00, K01, K010, K011, K012, K014, K02, K03, K04, K05, K06, K07, K08, K09, K11, K110, K111, K112, K114, K12, K13, K14, K15, K16, K17, K18, K19, K21, K210, K211, K214, K22, K23, K24, K25, K26, K27, K28, K29, K31, K310, K313, K314, K32, K33, K34, K35, K36, K37, K38, K39, K412, K413, K414: footprint keebs:Mx_Alps_100 -> Button_Switch_Keyboard:SW_Cherry_MX_1.00u_PCB; symbol keyboard_parts:KEYSW -> keyboard2-rescue:KEYSW-keyboard_parts
- K013: footprint keebs:Mx_Alps_100 -> Button_Switch_Keyboard:SW_Cherry_MX_2.00u_PCB; symbol keyboard_parts:KEYSW -> keyboard2-rescue:KEYSW-keyboard_parts
- K10, K113: footprint keebs:Mx_Alps_100 -> Button_Switch_Keyboard:SW_Cherry_MX_1.50u_PCB; symbol keyboard_parts:KEYSW -> keyboard2-rescue:KEYSW-keyboard_parts
- K20: footprint keebs:Mx_Alps_100 -> Button_Switch_Keyboard:SW_Cherry_MX_1.75u_PCB; symbol keyboard_parts:KEYSW -> keyboard2-rescue:KEYSW-keyboard_parts
- K212, K30: footprint keebs:Mx_Alps_100 -> Button_Switch_Keyboard:SW_Cherry_MX_2.25u_PCB; symbol keyboard_parts:KEYSW -> keyboard2-rescue:KEYSW-keyboard_parts
- K311: footprint keebs:Mx_Alps_100 -> Button_Switch_Keyboard:SW_Cherry_MX_2.75u_PCB; symbol keyboard_parts:KEYSW -> keyboard2-rescue:KEYSW-keyboard_parts
- K40, K41, K410, K411, K42, K49: footprint keebs:Mx_Alps_100 -> Button_Switch_Keyboard:SW_Cherry_MX_1.25u_PCB; symbol keyboard_parts:KEYSW -> keyboard2-rescue:KEYSW-keyboard_parts
- K45: footprint keebs:Mx_Alps_100 -> Button_Switch_Keyboard:SW_Cherry_MX_6.25u_PCB; symbol keyboard_parts:KEYSW -> keyboard2-rescue:KEYSW-keyboard_parts
Connections:
- net col8: now also K48.1
- net row4: now also D48.1 (K)
- new net: D48.2 (A), K48.2

Commit message: finished row wiring with new components
Parts:
- J1: footprint Connector_PinHeader_1.00mm:PinHeader_1x16_P1.00mm_Vertical -> Connector_PinHeader_2.54mm:PinHeader_1x16_P2.54mm_Vertical
- J2: footprint Connector_PinHeader_1.00mm:PinHeader_1x12_P1.00mm_Vertical -> Connector_PinHeader_2.54mm:PinHeader_1x12_P2.54mm_Vertical
Changed lines of the file:
@@
 F 0 "J2" H 10292 5575 50  0000 C CNN
 F 1 "Conn_01x12_Female" H 10292 5666 50  0000 C CNN
-F 2 "Connector_PinHeader_1.00mm:PinHeader_1x12_P1.00mm_Vertical" H 10400 6400 50  0001 C CNN
+F 2 "Connector_PinHeader_2.54mm:PinHeader_1x12_P2.54mm_Vertical" H 10400 6400 50  0001 C CNN
 F 3 "~" H 10400 6400 50  0001 C CNN
 	1    10400 6400
@@
 F 0 "J1" H 9750 6450 50  0000 L CNN
 F 1 "Conn_01x16_Female" V 9750 5600 50  0000 L CNN
-F 2 "Connector_PinHeader_1.00mm:PinHeader_1x16_P1.00mm_Vertical" H 9700 6300 50  0001 C CNN
+F 2 "Connector_PinHeader_2.54mm:PinHeader_1x16_P2.54mm_Vertical" H 9700 6300 50  0001 C CNN
 F 3 "~" H 9700 6300 50  0001 C CNN
 	1    9700 6300

Commit message: rev1 complete
Connections:
- net col0: now also J1.15 (Pin_15); no longer J1.10 (Pin_10)
- net col1: now also J1.14 (Pin_14); no longer J1.11 (Pin_11)
- net col2: now also J1.13 (Pin_13); no longer J1.12 (Pin_12)
- net col3: now also J1.12 (Pin_12); no longer J1.13 (Pin_13)
- net col4: now also J1.11 (Pin_11); no longer J1.14 (Pin_14)
- net col5: now also J1.10 (Pin_10); no longer J1.15 (Pin_15)
Changed lines of the file:
@@
 Wire Wire Line
 	9300 6400 9500 6400
+Text Label 9300 7000 0    50   ~ 0
+col0
+Text Label 9300 6900 0    50   ~ 0
+col1
+Text Label 9300 6800 0    50   ~ 0
+col2
+Text Label 9300 6700 0    50   ~ 0
+col3
+Text Label 9300 6600 0    50   ~ 0
+col4
 Text Label 9300 6500 0    50   ~ 0
-col0
-Text Label 9300 6600 0    50   ~ 0
-col1
-Text Label 9300 6700 0    50   ~ 0
-col2
-Text Label 9300 6800 0    50   ~ 0
-col3
-Text Label 9300 6900 0    50   ~ 0
-col4
-Text Label 9300 7000 0    50   ~ 0
 col5
 Text Label 10750 6100 0    50   ~ 0
