File: keyboard2.kicad_pcb (KiCad board)
At the start: 2 copper layers, 138 parts, among them J1 Conn_01x16_Female, J2 Conn_01x12_Female, K00 KEYSW, K01 KEYSW, K010 KEYSW, K011 KEYSW, K012 KEYSW, K013 KEYSW, K014 KEYSW, K02 KEYSW, K03 KEYSW, K04 KEYSW, K05 KEYSW, K06 KEYSW, K07 KEYSW, K08 KEYSW, K09 KEYSW, K10 KEYSW, K11 KEYSW, K110 KEYSW, K111 KEYSW, K112 KEYSW, K113 KEYSW, K114 KEYSW, K12 KEYSW, K13 KEYSW, K14 KEYSW, K15 KEYSW, K16 KEYSW, K17 KEYSW, K18 KEYSW, K19 KEYSW, K20 KEYSW, K21 KEYSW, K210 KEYSW, K211 KEYSW, K212 KEYSW, K214 KEYSW, K22 KEYSW, K23 KEYSW, K24 KEYSW, K25 KEYSW, K26 KEYSW, K27 KEYSW, K28 KEYSW, K29 KEYSW, K30 KEYSW, K31 KEYSW, K310 KEYSW, K311 KEYSW, K313 KEYSW, K314 KEYSW, K32 KEYSW, K33 KEYSW, K34 KEYSW, K35 KEYSW, K36 KEYSW, K37 KEYSW, K38 KEYSW, K39 KEYSW, K40 KEYSW, K41 KEYSW, K410 KEYSW, K411 KEYSW, K412 KEYSW, K413 KEYSW, K414 KEYSW, K42 KEYSW, K45 KEYSW, K49 KEYSW

Commit message: finished basic layout iteration 1
Parts:
- moved K313 368.1 mm to (331.0, 79.4)
- moved K414 349.6 mm to (350.0, 98.4)
- moved K212 349.0 mm to (276.2, 60.3)
- moved K413 339.6 mm to (331.0, 98.4)
- moved K314 338.8 mm to (350.0, 41.3)
- moved K214 306.4 mm to (331.0, 41.3)
- moved K211 298.9 mm to (245.3, 60.3)
- moved K27 298.9 mm to (169.1, 60.3)
- moved K411 296.2 mm to (270.7, 98.4)
- moved K412 295.9 mm to (311.9, 98.4)
- moved K311 291.7 mm to (271.5, 79.4)
- moved K20 284.2 mm to (28.6, 60.3)
- moved K34 271.9 mm to (121.4, 79.4)
- moved K39 269.1 mm to (216.7, 79.4)
- moved K26 268.0 mm to (150.0, 60.3)
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
Commit message: start work on traces
Parts:
- moved D014 406.7 mm to (331.0, 27.0)
- moved D012 394.9 mm to (250.8, 27.0)
- moved D00 385.7 mm to (22.2, 27.0)
- moved D03 381.4 mm to (79.4, 27.0)
- moved D01 368.9 mm to (41.3, 27.0)
- moved D011 367.9 mm to (231.5, 27.0)
- moved D20 366.6 mm to (28.6, 65.1)
- moved D05 357.6 mm to (117.5, 27.0)
- moved D110 356.4 mm to (222.2, 46.0)
- moved D10 354.2 mm to (27.0, 46.0)
- moved D02 353.7 mm to (60.3, 27.0)
- moved D21 351.1 mm to (54.8, 65.1)
- moved D212 348.3 mm to (276.2, 65.1)
- moved D010 344.6 mm to (212.7, 27.0)
- moved D14 344.3 mm to (108.0, 46.0)
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Routing:
- net /row1: track 0.00 -> 426.0 mm
- net /row0: track 0.00 -> 413.1 mm
Other:
- board outline added: 355.6 x 103.2 mm

Commit message: finished row traces
Parts:
- moved J2 1.11 mm to (314.0, 64.0)
- moved J1 0.30 mm to (293.7, 60.0)
Routing:
- net /row3: track 0.00 -> 488.7 mm
- net /row2: track 0.00 -> 424.3 mm
- net /row4: track 0.00 -> 381.9 mm
- net /row1: track 426.0 -> 446.9 mm

Commit message: used the wrong diodes, have to redo all traces
Parts:
- D00: footprint keyboard_parts:D_SOD123_axial -> Diode_SMD:D_SOD-123
Routing:
- net /row3: track 488.7 -> 0.00 mm
- net /row1: track 446.9 -> 0.00 mm
- net /row2: track 424.3 -> 0.00 mm
- net /row0: track 413.0 -> 0.00 mm
- net /row4: track 381.9 -> 0.00 mm

Commit message: finished alphanumeric placement on pcb
Parts:
- added D48: D, Diode_SMD:D_SOD-123, F.Cu at (78.6, 293.6)
- added K48: KEYSW, Button_Switch_Keyboard:SW_Cherry_MX_1.25u_PCB, F.Cu at (216.8, 92.5)
- D01, D010, D011, D012, D013, D014, D02, D03, D04, D05, D06, D07, D08, D09, D10, D11, D110, D111, D112, D113, D114, D12, D13, D14, D15, D16, D17, D18, D19, D20, D21, D210, D211, D212, D214, D22, D23, D24, D25, D26, D27, D28, D29, D30, D31, D310, D311, D313, D314, D32, D33, D34, D35, D36, D37, D38, D39, D40, D41, D410, D411, D412, D413, D414, D42, D45, D49: footprint keyboard_parts:D_SOD123_axial -> Diode_SMD:D_SOD-123
- K00, K01, K010, K011, K012, K014, K02, K03, K04, K05, K06, K07, K08, K09, K11, K110, K111, K112, K114, K12, K13, K14, K15, K16, K17, K18, K19, K21, K210, K211, K214, K22, K23, K24, K25, K26, K27, K28, K29, K31, K310, K313, K314, K32, K33, K34, K35, K36, K37, K38, K39, K412, K413, K414: footprint keebs:Mx_Alps_100 -> Button_Switch_Keyboard:SW_Cherry_MX_1.00u_PCB
- K013: footprint keebs:Mx_Alps_100 -> Button_Switch_Keyboard:SW_Cherry_MX_2.00u_PCB
- K10, K113: footprint keebs:Mx_Alps_100 -> Button_Switch_Keyboard:SW_Cherry_MX_1.50u_PCB
- K20: footprint keebs:Mx_Alps_100 -> Button_Switch_Keyboard:SW_Cherry_MX_1.75u_PCB
- K212, K30: footprint keebs:Mx_Alps_100 -> Button_Switch_Keyboard:SW_Cherry_MX_2.25u_PCB
- K311: footprint keebs:Mx_Alps_100 -> Button_Switch_Keyboard:SW_Cherry_MX_2.75u_PCB
- K40, K41, K410, K411, K42, K49: footprint keebs:Mx_Alps_100 -> Button_Switch_Keyboard:SW_Cherry_MX_1.25u_PCB
- K45: footprint keebs:Mx_Alps_100 -> Button_Switch_Keyboard:SW_Cherry_MX_6.25u_PCB
- moved D114 486.9 mm to (43.0, 404.8)
- moved D314 483.6 mm to (25.8, 404.8)
- moved D214 469.9 mm to (31.5, 408.2)
- moved D414 453.6 mm to (14.3, 408.2)
- moved D113 448.8 mm to (14.3, 404.8)
- moved D014 445.6 mm to (94.8, 404.8)
- moved D313 433.5 mm to (43.0, 408.2)
- moved D413 433.2 mm to (20.0, 404.8)
- moved D212 427.5 mm to (25.8, 411.5)
- moved D112 425.5 mm to (31.5, 404.8)
- moved D412 422.2 mm to (20.0, 408.2)
- moved D013 419.4 mm to (112.0, 411.5)
- moved D011 408.1 mm to (94.8, 411.5)
- moved D211 407.1 mm to (31.5, 411.5)
- moved D012 404.5 mm to (106.3, 404.8)
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Other:
- board outline removed

Commit message: finished row wiring with new components
Parts:
- J1: footprint Connector_PinHeader_1.00mm:PinHeader_1x16_P1.00mm_Vertical -> Connector_PinHeader_2.54mm:PinHeader_1x16_P2.54mm_Vertical
- J2: footprint Connector_PinHeader_1.00mm:PinHeader_1x12_P1.00mm_Vertical -> Connector_PinHeader_2.54mm:PinHeader_1x12_P2.54mm_Vertical
- moved D214 496.8 mm to (354.8, 31.0)
- moved D314 477.8 mm to (345.6, 49.9)
- moved D114 474.8 mm to (335.7, 31.0)
- moved D414 454.5 mm to (354.8, 107.1)
- moved D113 445.3 mm to (283.4, 50.0)
- moved D413 433.9 mm to (335.7, 107.1)
- moved D313 433.7 mm to (335.7, 88.1)
- moved D014 430.0 mm to (307.2, 31.0)
- moved D212 424.3 mm to (276.2, 69.1)
- moved D412 422.6 mm to (316.7, 107.1)
- moved D112 421.8 mm to (259.5, 50.0)
- moved D013 415.4 mm to (278.6, 31.0)
- moved D411 407.8 mm to (285.7, 107.1)
- moved D011 404.2 mm to (231.0, 31.0)
- moved D211 403.7 mm to (245.3, 69.1)
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Routing:
- net /row4: track 0.00 -> 399.1 mm
- net /row2: track 0.00 -> 375.6 mm
- net /row3: track 0.00 -> 362.2 mm
- net /row1: track 0.00 -> 354.6 mm
- net /row0: track 0.00 -> 327.1 mm
- net Net-(D413-Pad2): track 0.00 -> 14.3 mm
- net Net-(D410-Pad2): track 0.00 -> 14.3 mm
- net Net-(D313-Pad2): track 0.00 -> 14.3 mm
- net Net-(D112-Pad2): track 0.00 -> 14.3 mm
- net Net-(D214-Pad2): track 0.00 -> 14.3 mm
- net Net-(D29-Pad2): track 0.00 -> 14.3 mm
- net Net-(D28-Pad2): track 0.00 -> 14.3 mm
- net Net-(D27-Pad2): track 0.00 -> 14.3 mm
- net Net-(D26-Pad2): track 0.00 -> 14.3 mm
- net Net-(D25-Pad2): track 0.00 -> 14.3 mm
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Other:
- board outline added: 356.4 x 102.4 mm

Commit message: rev1 complete
Connections:
- J1 pad 10: /col0 -> /col5
- J1 pad 11: /col1 -> /col4
- J1 pad 12: /col2 -> /col3
- J1 pad 13: /col3 -> /col2
- J1 pad 14: /col4 -> /col1
- J1 pad 15: /col5 -> /col0
Routing:
- net /col0: track 0.00 -> 419.1 mm
- net /col1: track 0.00 -> 391.2 mm
- net /col2: track 0.00 -> 369.7 mm
- net /col3: track 0.00 -> 338.1 mm
- net /col4: track 0.00 -> 321.0 mm
- net /col5: track 0.00 -> 306.8 mm
- net /col6: track 0.00 -> 305.5 mm
- net /col7: track 0.00 -> 292.1 mm
- net /col8: track 0.00 -> 283.3 mm
- net /col9: track 0.00 -> 245.2 mm
- net /col10: track 0.00 -> 233.5 mm
- net /col11: track 0.00 -> 185.6 mm
- net /col14: track 0.00 -> 171.9 mm
- net /col12: track 0.00 -> 156.7 mm
- net /col13: track 0.00 -> 148.6 mm
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